Commit message: Add capability to switch hardware interface to allow velocity controller

File: ur_description/urdf/inc/ur_macro.xacro (robot description, xacro)
@@ -50,5 +50,6 @@
     physical_parameters_file
     visual_parameters_file
-    transmission_hw_interface:=hardware_interface/PositionJointInterface
+    hw_interface_1:=hardware_interface/PositionJointInterface
+    hw_interface_2:=hardware_interface/VelocityJointInterface
     safety_limits:=false
     safety_pos_margin:=0.15
@@ -62,5 +63,5 @@
       visual_parameters_file="${visual_parameters_file}"/>
     <!-- Add URDF transmission elements (for ros_control) -->
-    <xacro:ur_arm_transmission prefix="${prefix}" hw_interface="${transmission_hw_interface}" />
+    <xacro:ur_arm_transmission prefix="${prefix}" hw_interface_1="${hw_interface_1}" hw_interface_2="${hw_interface_2}"/>
     <!-- links: main serial chain -->
     <link name="${prefix}base_link"/>

File: ur_description/urdf/inc/ur_transmissions.xacro (robot description, xacro)
@@ -6,9 +6,10 @@
           this location. Nor can they rely on the existence of the macro.
   -->
-  <xacro:macro name="ur_arm_transmission" params="prefix hw_interface">
+  <xacro:macro name="ur_arm_transmission" params="prefix hw_interface_1 hw_interface_2">
     <transmission name="${prefix}shoulder_pan_trans">
       <type>transmission_interface/SimpleTransmission</type>
       <joint name="${prefix}shoulder_pan_joint">
-        <hardwareInterface>${hw_interface}</hardwareInterface>
+        <hardwareInterface>${hw_interface_1}</hardwareInterface>
+	<hardwareInterface>${hw_interface_2}</hardwareInterface>
       </joint>
       <actuator name="${prefix}shoulder_pan_motor">
@@ -19,5 +20,6 @@
       <type>transmission_interface/SimpleTransmission</type>
       <joint name="${prefix}shoulder_lift_joint">
-        <hardwareInterface>${hw_interface}</hardwareInterface>
+        <hardwareInterface>${hw_interface_1}</hardwareInterface>
+        <hardwareInterface>${hw_interface_2}</hardwareInterface>
       </joint>
       <actuator name="${prefix}shoulder_lift_motor">
@@ -28,5 +30,6 @@
       <type>transmission_interface/SimpleTransmission</type>
       <joint name="${prefix}elbow_joint">
-        <hardwareInterface>${hw_interface}</hardwareInterface>
+        <hardwareInterface>${hw_interface_1}</hardwareInterface>
+        <hardwareInterface>${hw_interface_2}</hardwareInterface>
       </joint>
       <actuator name="${prefix}elbow_motor">
@@ -37,5 +40,6 @@
       <type>transmission_interface/SimpleTransmission</type>
       <joint name="${prefix}wrist_1_joint">
-        <hardwareInterface>${hw_interface}</hardwareInterface>
+        <hardwareInterface>${hw_interface_1}</hardwareInterface>
+        <hardwareInterface>${hw_interface_2}</hardwareInterface>
       </joint>
       <actuator name="${prefix}wrist_1_motor">
@@ -46,5 +50,6 @@
       <type>transmission_interface/SimpleTransmission</type>
       <joint name="${prefix}wrist_2_joint">
-        <hardwareInterface>${hw_interface}</hardwareInterface>
+        <hardwareInterface>${hw_interface_1}</hardwareInterface>
+        <hardwareInterface>${hw_interface_2}</hardwareInterface>
       </joint>
       <actuator name="${prefix}wrist_2_motor">
@@ -55,5 +60,6 @@
       <type>transmission_interface/SimpleTransmission</type>
       <joint name="${prefix}wrist_3_joint">
-        <hardwareInterface>${hw_interface}</hardwareInterface>
+        <hardwareInterface>${hw_interface_1}</hardwareInterface>
+        <hardwareInterface>${hw_interface_2}</hardwareInterface>
       </joint>
       <actuator name="${prefix}wrist_3_motor">

File: ur_gazebo/urdf/ur.xacro (robot description, xacro)
@@ -38,5 +38,6 @@
           controller .yaml files in the 'config' directory.
   -->
-  <xacro:arg name="transmission_hw_interface" default="hardware_interface/PositionJointInterface"/>
+  <xacro:arg name="transmission_hw_interface_1" default="hardware_interface/PositionJointInterface"/>
+  <xacro:arg name="transmission_hw_interface_2" default="hardware_interface/VelocityJointInterface"/>
   <xacro:arg name="safety_limits" default="false"/>
   <xacro:arg name="safety_pos_margin" default="0.15"/>
@@ -50,4 +51,6 @@
     visual_parameters_file="$(arg visual_params)"
     transmission_hw_interface="$(arg transmission_hw_interface)"
+    transmission_hw_interface_1="$(arg transmission_hw_interface_1)"
+    transmission_hw_interface_2="$(arg transmission_hw_interface_2)"
     safety_limits="$(arg safety_limits)"
     safety_pos_margin="$(arg safety_pos_margin)"

File: ur_gazebo/urdf/ur_macro.xacro (robot description, xacro)
@@ -37,5 +37,6 @@
    physical_parameters_file
    visual_parameters_file
-   transmission_hw_interface:=hardware_interface/PositionJointInterface
+   transmission_hw_interface_1:=hardware_interface/PositionJointInterface
+   transmission_hw_interface_2:=hardware_interface/VelocityJointInterface
    safety_limits:=false safety_pos_margin:=0.15 safety_k_position:=20"
   >
@@ -54,5 +55,6 @@
       physical_parameters_file="${physical_parameters_file}"
       visual_parameters_file="${visual_parameters_file}"
-      transmission_hw_interface="${transmission_hw_interface}"
+      hw_interface_1="${transmission_hw_interface_1}"
+      interface_2="${transmission_hw_interface_2}"
       safety_limits="${safety_limits}"
       safety_pos_margin="${safety_pos_margin}"
@@ -62,22 +64,29 @@
     <gazebo reference="${prefix}shoulder_link">
       <selfCollide>true</selfCollide>
+      <turnGravityOff>true</turnGravityOff>
     </gazebo>
     <gazebo reference="${prefix}upper_arm_link">
       <selfCollide>true</selfCollide>
+      <turnGravityOff>true</turnGravityOff>
     </gazebo>
     <gazebo reference="${prefix}forearm_link">
       <selfCollide>true</selfCollide>
+      <turnGravityOff>true</turnGravityOff>
     </gazebo>
     <gazebo reference="${prefix}wrist_1_link">
       <selfCollide>true</selfCollide>
+      <turnGravityOff>true</turnGravityOff>
     </gazebo>
     <gazebo reference="${prefix}wrist_3_link">
       <selfCollide>true</selfCollide>
+      <turnGravityOff>true</turnGravityOff>
     </gazebo>
     <gazebo reference="${prefix}wrist_2_link">
       <selfCollide>true</selfCollide>
+      <turnGravityOff>true</turnGravityOff>
     </gazebo>
     <gazebo reference="${prefix}ee_link">
       <selfCollide>true</selfCollide>
+      <turnGravityOff>true</turnGravityOff>
     </gazebo>
     <!--
@@ -86,7 +95,8 @@
     -->
     <gazebo>
-      <plugin name="ros_control" filename="libgazebo_ros_control.so">
+      <plugin name="cob_gazebo_ros_control" filename="libhwi_switch_gazebo_ros_control.so">
         <!--robotNamespace>/</robotNamespace-->
         <!--robotSimType>gazebo_ros_control/DefaultRobotHWSim</robotSimType-->
+        <robotSimType>cob_gazebo_ros_control/HWISwitchRobotHWSim</robotSimType>
       </plugin>
     </gazebo>
